File: mora-jai.kicad_sch (KiCad schematic)
At the start: 0 parts

Commit message: lay out MCU, buttons, mux, and some initial LEDs in schematic
Parts:
- added SW1, SW10, SW11, SW12, SW13, SW14, SW15, SW16, SW2, SW3, SW4, SW5, SW6, SW7, SW8, SW9: SW_Push, symbol Switch:SW_Push
- added U1: CD74HC4067M, Package_SO:SOIC-24W_7.5x15.4mm_P1.27mm, symbol 74xx:CD74HC4067M
- added U2: XIAO-ESP32-S3-DIP, Module:MOUDLE14P-XIAO-DIP-SMD, symbol Seeed_Studio_XIAO_Series:XIAO-ESP32-S3-DIP
Connections:
- new net +3V3: U2.12 (VCC_3V3)
- new net +5V: U1.24 (VCC), U2.14 (VBUS)
- new net COPI: U2.11 (GPIO9/D10/A10/MOSI)
- new net GND: U1.12 (GND), U2.13 (GND)
- new net MUX_EN: U1.15 (~{E})
- new net PICO: U2.10 (GPIO8/D9/A9/MISO)
- new net SCL: U2.6 (GPIO9/D5/I2C_SCL)
- new net SDA: U2.5 (GPIO5/D4/I2C_SDA)
- new net SW_0: U1.9 (I0)
- new net SW_1: U1.8 (I1)
- new net SW_10: U1.21 (I10)
- new net SW_11: U1.20 (I11)
- new net SW_12: U1.19 (I12)
- new net SW_13: U1.18 (I13)
- new net SW_14: U1.17 (I14)
- new net SW_15: U1.16 (I15)
- new net SW_2: U1.7 (I2)
- new net SW_3: U1.6 (I3)
- new net SW_4: U1.5 (I4)
- new net SW_5: U1.4 (I5)
- new net SW_6: U1.3 (I6)
- new net SW_7: U1.2 (I7)
- new net SW_8: U1.23 (I8)
- new net SW_9: U1.22 (I9)
- no-connect marks 0 -> 3
Other:
- added sheet LED matrix (led_matrix.kicad_sch)
