File: pcb/led_matrix.kicad_sch (KiCad schematic)
At the start: 44 parts

Commit message: placing power components
Other:
- note removed: "Questions: - Is one LED per corner acceptable?"
Changed lines of the file:
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@@
-		)
-	)
-	(text "Questions:\n- Is one LED per corner acceptable?"
-		(exclude_from_sim no)
-		(at 126.746 152.4 0)
-		(effects
-			(font
-				(size 1.524 1.524)
-			)
-			(justify left)
 		)
 	)
