File: pcb/power.kicad_sch (KiCad schematic)
At the start: 22 parts, among them IC1 TPS61023DRLR, Q1 Q_PMOS_DGS, U2 MCP73833-AMI-UN

Commit message: placing power components
Parts:
- added J1: Conn_01x02, Connector_JST:JST_PH_S2B-PH-K_1x02_P2.00mm_Horizontal, symbol Connector_Generic:Conn_01x02
- added J10: Conn_01x04, Connector_PinSocket_2.54mm:PinSocket_1x04_P2.54mm_Vertical, symbol Connector_Generic:Conn_01x04
- added J3, J6, J7, J8: Conn_01x02, Connector_PinSocket_2.54mm:PinSocket_1x02_P2.54mm_Vertical, symbol Connector_Generic:Conn_01x02
- added J4: Conn_01x03, Connector_PinSocket_2.54mm:PinSocket_1x03_P2.54mm_Vertical, symbol Connector_Generic:Conn_01x03
- added S1: SLW-874744-6A-RA-N-D, Mora_Jai_Parts:SW_SLW-874744-6A-RA-N-D, symbol Mora_Jai_Sym:SLW-874744-6A-RA-N-D
- D5: footprint (none) -> Diode_SMD:D_SOD-123F
- L1: footprint (none) -> Mora_Jai_Parts:74438356010
- Q1: footprint (none) -> Package_TO_SOT_SMD:SOT-323_SC-70
Connections:
- net +3V3: now also J6.1 (Pin_1)
- net +5V: now also J3.1 (Pin_1), S1.1; no longer C28.1, C30.1, IC1.6 (VOUT), R11.1
- net +BATT: now also J1.1 (Pin_1)
- net GND: now also J1.2 (Pin_2), J10.4 (Pin_4), J3.2 (Pin_2), J6.2 (Pin_2), J7.2 (Pin_2), J8.2 (Pin_2), S1.SH1, S1.SH2
- net VBUS: now also J10.1 (Pin_1)
- net VIN: now also J7.1 (Pin_1)
- net ~{PWR_GOOD}: now also J4.3 (Pin_3)
- net ~{STAT1}: now also J4.1 (Pin_1)
- net ~{STAT2}: now also J4.2 (Pin_2)
- new net USB_D+: J10.2 (Pin_2)
- new net USB_D-: J10.3 (Pin_3)
- new net V_OUT: C28.1, C30.1, IC1.6 (VOUT), J8.1 (Pin_1), R11.1, S1.2
- no-connect marks 0 -> 1
Other:
- note added: "+5V Boost converter"
- note added: "Battery connector"
- note added: "Differential routing for data traces!!"
- note added: "Power Test Pads"
- note added: "Power switch"
- note added: "USB wire breakout"
- note added: "charger status indicators"
- note removed: "TODO: check where this should be connected"
- moved on the sheet: C20, C26, D5, Q1, R10, R3, R9

Commit message: drew fill zones for battery charger
Changed lines of the file:
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@@
+	)
+	(junction
+		(at 167.64 43.18)
+		(diameter 0)
+		(color 0 0 0 0)
 	)
 	(junction
@@
 	(wire
 		(pts
-			(xy 154.94 43.18) (xy 172.72 43.18)
+			(xy 154.94 43.18) (xy 167.64 43.18)
 		)
 		(stroke
@@
 	(wire
 		(pts
+			(xy 167.64 43.18) (xy 172.72 43.18)
+		)
+		(stroke
+			(width 0)
+			(type default)
+		)
+	)
+	(wire
+		(pts
 			(xy 39.37 93.98) (xy 39.37 92.71)
 		)
@@
 	(wire
 		(pts
+			(xy 119.38 109.22) (xy 121.92 109.22)
+		)
+		(stroke
+			(width 0)
+			(type default)
+		)
+	)
+	(wire
+		(pts
 			(xy 172.72 64.77) (xy 172.72 67.31)
 		)
@@
 	(wire
 		(pts
+			(xy 167.64 44.45) (xy 167.64 43.18)
+		)
+		(stroke
+			(width 0)
+			(type default)
+		)
+	)
+	(wire
+		(pts
 			(xy 154.94 43.18) (xy 146.05 43.18)
 		)
@@
 	(wire
 		(pts
-			(xy 116.84 109.22) (xy 121.92 109.22)
-		)
-		(stroke
-			(width 0)
-			(type default)
-		)
-	)
-	(wire
-		(pts
 			(xy 104.14 85.09) (xy 96.52 85.09)
 		)
@@
 			(width 0)
 			(type default)
-		)
-	)
-	(label "VIN"
-		(at 116.84 109.22 0)
-		(effects
-			(font
-				(size 1.27 1.27)
-			)
-			(justify left bottom)
-		)
-	)
-	(label "VIN"
-		(at 162.56 43.18 0)
-		(effects
-			(font
-				(size 1.27 1.27)
-			)
-			(justify left bottom)
 		)
 	)
@@
 		)
 	)
+	(global_label "VIN"
+		(shape input)
+		(at 119.38 109.22 180)
+		(fields_autoplaced yes)
+		(effects
+			(font
+				(size 1.27 1.27)
+			)
+			(justify right)
+		)
+		(property "Intersheetrefs" "${INTERSHEET_REFS}"
+			(at 113.3709 109.22 0)
+			(hide yes)
+			(show_name no)
+			(do_not_autoplace no)
+			(effects
+				(font
+					(size 1.27 1.27)
+				)
+				(justify right)
+			)
+		)
+	)
 	(global_label "V_OUT"
 		(shape input)
@@
 			(hide yes)
 			(show_name no)
+			(do_not_autoplace no)
+			(effects
+				(font
+					(size 1.27 1.27)
+				)
+				(justify right)
+			)
+		)
+	)
+	(global_label "VIN"
+		(shape input)
+		(at 167.64 44.45 270)
+		(fields_autoplaced yes)
+		(effects
+			(font
+				(size 1.27 1.27)
+			)
+			(justify right)
+		)
+		(property "Intersheetrefs" "${INTERSHEET_REFS}"
+			(at 167.64 50.4591 90)
+			(hide yes)
+			(show_name no)
